File: psd_bus.kicad_pcb (KiCad board)
At the start: 2 copper layers, 112.4 x 105.5 mm, 35 parts, among them J1 PMOD1, J10 PMOD2, J11 RASPBERRYPI_BPLUS_BONNETNODIM, J12 Conn_02x20_Odd_Even, J13 PMOD3, J14 DINC_MIN_TM_6_1, J15 USB3_A, J16 Conn_01x06, J17 Conn_01x03, J2 Conn_02x40_Odd_Even, J9 Conn_01x02

Commit message: preliminary distribution on pcb
Parts:
- removed JP11: Conn_01x03, Connector_PinHeader_2.54mm:PinHeader_1x03_P2.54mm_Vertical
- removed LO2: OSHW-Logo2_14.6x12mm_SilkScreen, Symbol:OSHW-Logo2_14.6x12mm_SilkScreen
- removed R11, R12, R13: 510, Resistor_SMD:R_0805_2012Metric_Pad1.20x1.40mm_HandSolder
- added BUT1: SW_DIP_x01, Button_Switch_THT:SW_PUSH_6mm_H5mm, F.Cu at (110.3, 56.5)
- added BUT2: SW_DIP_x01, Button_Switch_THT:SW_PUSH_6mm_H5mm, F.Cu at (126.3, 56.2)
- added C1: 1uF, Capacitor_SMD:C_0805_2012Metric_Pad1.18x1.45mm_HandSolder, F.Cu at (81.3, 97.2)
- added C2: 10uF, Capacitor_SMD:C_0805_2012Metric_Pad1.18x1.45mm_HandSolder, F.Cu at (101.9, 113.1)
- added C4: 100nF, Capacitor_SMD:C_0603_1608Metric, F.Cu at (73.5, 87.8)
- added D5: LED, LED_SMD:LED_0805_2012Metric_Pad1.15x1.40mm_HandSolder, F.Cu at (142.0, 82.7)
- added D6: LED, LED_SMD:LED_0805_2012Metric_Pad1.15x1.40mm_HandSolder, F.Cu at (150.1, 75.5)
- added D7: LED, LED_SMD:LED_0805_2012Metric_Pad1.15x1.40mm_HandSolder, F.Cu at (150.1, 83.2)
- added J18: DINC_MIN_TM_6_1, footprints:DINC_MIN_TM_6_1PRIMARY, F.Cu at (67.3, 127.0)
- added J19: Conn_02x06_Odd_Even, Connector_PinSocket_2.54mm:PinSocket_1x06_P2.54mm_Vertical, F.Cu at (62.2, 68.6)
- added J20: USB3_A, footprints:USB-3.0-TH_C69073, F.Cu at (160.0, 114.3)
- added J21: DB9_Male_MountingHoles, Connector_Dsub:DSUB-9_Male_Horizontal_P2.77x2.84mm_EdgePinOffset9.90mm_Housed_MountingHolesOffset11.32mm, F.Cu at (120.2, 114.8)
- added J3: PMOD4, footprints:PMOD_Female_Horizontal_2, F.Cu at (153.1, 36.4)
- added J4: Conn_02x20_Odd_Even, Connector_PinHeader_2.54mm:PinHeader_2x20_P2.54mm_Vertical, F.Cu at (50.8, 74.9)
- added J5: Conn_01x03, Connector_PinSocket_2.54mm:PinSocket_1x03_P2.54mm_Vertical, F.Cu at (44.5, 116.9)
- added J6: Conn_01x02, Connector_PinSocket_2.54mm:PinSocket_1x02_P2.54mm_Vertical, F.Cu at (135.9, 33.7)
- added J7: Conn_01x05, Connector_PinSocket_2.54mm:PinSocket_1x05_P2.54mm_Vertical, F.Cu at (52.8, 35.5)
- added J8: Conn_01x04, footprints:I2C_DISPLAY_MULTI2, F.Cu at (125.7, 104.1)
- added JP1: Conn_01x02, Connector_PinHeader_2.54mm:PinHeader_1x02_P2.54mm_Vertical, F.Cu at (61.0, 87.6)
- added JP2: Conn_01x02, Connector_PinHeader_2.54mm:PinHeader_1x02_P2.54mm_Vertical, F.Cu at (61.0, 106.7)
- added JP3: Conn_01x02, Connector_PinHeader_2.54mm:PinHeader_1x02_P2.54mm_Vertical, F.Cu at (84.5, 46.4)
- added JP4: Conn_01x02, Connector_PinHeader_2.54mm:PinHeader_1x02_P2.54mm_Vertical, F.Cu at (62.9, 46.4)
- added JP6: Conn_01x03, Connector_PinHeader_2.54mm:PinHeader_1x03_P2.54mm_Vertical, F.Cu at (144.1, 94.0)
- added JP8: Conn_01x03, Connector_PinHeader_2.54mm:PinHeader_1x03_P2.54mm_Vertical, F.Cu at (141.0, 102.9)
- added JPS1: SolderJumper_3_Open, Jumper:SolderJumper-3_P1.3mm_Open_RoundedPad1.0x1.5mm_NumberLabels, F.Cu at (78.1, 109.2)
- added JPS2: SolderJumper_3_Open, Jumper:SolderJumper-3_P1.3mm_Open_RoundedPad1.0x1.5mm_NumberLabels, F.Cu at (151.8, 56.7)
- added P1: MEM1055-00-280-01-B, Connector_Card:SD_TE_2041021, F.Cu at (175.3, 55.9)
- added R14: 510, Resistor_SMD:R_0805_2012Metric_Pad1.20x1.40mm_HandSolder, F.Cu at (142.0, 75.1)
- added R15: 510, Resistor_SMD:R_0805_2012Metric_Pad1.20x1.40mm_HandSolder, F.Cu at (142.1, 64.2)
- added R16: 510, Resistor_SMD:R_0805_2012Metric_Pad1.20x1.40mm_HandSolder, F.Cu at (148.0, 50.2)
- added R17: 510, Resistor_SMD:R_0805_2012Metric_Pad1.20x1.40mm_HandSolder, F.Cu at (142.1, 67.2)
- added R18: 510, Resistor_SMD:R_0805_2012Metric_Pad1.20x1.40mm_HandSolder, F.Cu at (106.7, 113.0)
- added R19: 510, Resistor_SMD:R_0805_2012Metric_Pad1.20x1.40mm_HandSolder, F.Cu at (151.1, 65.4)
- added R20: 510, Resistor_SMD:R_0805_2012Metric_Pad1.20x1.40mm_HandSolder, F.Cu at (76.2, 85.1)
- added R21: 510, Resistor_SMD:R_0805_2012Metric_Pad1.20x1.40mm_HandSolder, F.Cu at (101.9, 116.0)
- added R22: 510, Resistor_SMD:R_0805_2012Metric_Pad1.20x1.40mm_HandSolder, F.Cu at (76.3, 93.2)
- added RN2: 20K, Resistor_SMD:R_Array_Concave_4x0603, F.Cu at (158.8, 76.6)
- added RN3: 20K, Resistor_SMD:R_Array_Concave_4x0603, F.Cu at (154.5, 76.3)
- added U1: LM1117-3.3, Package_TO_SOT_SMD:SOT-223-3_TabPin2, F.Cu at (68.6, 76.2)
- added U2: TXS0108EPWR, Package_SO:TSSOP-20_4.4x6.5mm_P0.65mm, F.Cu at (158.8, 92.7)
- J15: value USB3_A -> Conn_01x06; footprint footprints:USB-3.0-TH_C69073 -> footprints:PCM5102
- J16: value Conn_01x06 -> PMOD5; footprint Connector_PinSocket_2.54mm:PinSocket_1x06_P2.54mm_Vertical -> footprints:PMOD_Female_Horizontal_2
- R10: value 510 -> 200
- R5, R6: value 510 -> 1k
- R7, R8, R9: value 510 -> 220
- moved H3 125.3 mm to (157.5, 43.2)
- moved R6 98.4 mm to (148.0, 47.2)
- moved D4 97.5 mm to (142.6, 61.1)
- moved H1 96.3 mm to (69.2, 43.2)
- moved J16 92.0 mm to (174.0, 36.2)
- moved J14 91.0 mm to (85.9, 127.3), turned to 180 degrees
- moved J13 82.4 mm to (131.4, 36.1), turned to -90 degrees
- moved J1 81.8 mm to (85.7, 36.1), turned to -90 degrees
- moved J9 79.3 mm to (90.8, 36.1), turned to 180 degrees
- moved R8 78.0 mm to (143.3, 55.1)
- moved R7 77.8 mm to (151.3, 60.0)
- moved J10 75.5 mm to (108.6, 36.1), turned to -90 degrees
- moved JP12 67.1 mm to (114.3, 42.5), turned to 180 degrees
- moved R2 66.2 mm to (87.0, 109.2), turned to 90 degrees
- moved D2 65.9 mm to (90.8, 110.2), turned to 90 degrees
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Connections:
- D1 pad 1: /DETO5 -> /IO_50
- D2 pad 1: /DETO6 -> /IO_51
- D3 pad 1: /DETO3 -> /IO_52
- D4 pad 1: /DETO4 -> /IO_53
- J1 pad 1: /RGB_R2 -> /IO_1
- J1 pad 10: /RGB_B5 -> /IO_8
- J1 pad 2: /RGB_R3 -> /IO_2
- J1 pad 3: /RGB_R4 -> /IO_3
- J1 pad 4: /RGB_R5 -> /IO_4
- J1 pad 7: /RGB_B2 -> /IO_5
- J1 pad 8: /RGB_B3 -> /IO_6
- J1 pad 9: /RGB_B4 -> /IO_7
- J10 pad 1: /RGB_G2 -> /IO_9
- J10 pad 10: /DETO6 -> /IO_16
- J10 pad 2: /RGB_G3 -> /IO_10
- J10 pad 3: /RGB_G4 -> /IO_11
- J10 pad 4: /RGB_G5 -> /IO_12
- J10 pad 7: /HSYNC -> /IO_13
- J10 pad 8: /VSYNC -> /IO_14
- J10 pad 9: /DETO5 -> /IO_15
- J11 pad 1: /3V3pi -> unconnected-(J11-Pad1)
- J11 pad 10: /FPGA_Tx -> /IO_65
- J11 pad 11: /USER_IO2 -> /IO_57
- J11 pad 12: /AUDIO_IN -> /IO_66
- J11 pad 13: /USER_IO4 -> /IO_58
- J11 pad 15: /DETO2 -> /IO_59
- J11 pad 16: /DETO1 -> /IO_67
- J11 pad 17: /3V3pi -> unconnected-(J11-Pad1)
- J11 pad 18: /DETO3 -> /IO_68
- J11 pad 19: /MOSI -> /IO_60
- J11 pad 2: /5Vpi -> unconnected-(J11-Pad2)
- J11 pad 21: /MISO -> /IO_61
- J11 pad 22: /DETO4 -> /IO_69
- J11 pad 23: /SCK -> /IO_62
- J11 pad 24: /SS2_FPGA -> /IO_70
- J11 pad 29: /TMS -> unconnected-(J11-Pad29)
- J11 pad 3: /USER_IO1 -> /IO_54
- J11 pad 31: /LED_Y -> unconnected-(J11-Pad31)
- J11 pad 32: /TDI -> unconnected-(J11-Pad32)
- J11 pad 35: /DETO5 -> /IO_63
- J11 pad 36: /TDO -> unconnected-(J11-Pad36)
- J11 pad 38: /TCK -> unconnected-(J11-Pad38)
- J11 pad 4: /5Vpi -> unconnected-(J11-Pad2)
- J11 pad 40: /DETO6 -> /IO_71
- J11 pad 5: /USER_IO0 -> /IO_55
- J11 pad 7: unconnected-(J11-Pad7) -> /IO_56
- J11 pad 8: unconnected-(J11-Pad8) -> /IO_64
- J12 pad 1: /DETO5 -> /IO_50
- J12 pad 10: /USER_IO0 -> /IO_43
- J12 pad 11: /5Vmi -> Net-(J12-Pad11)
- J12 pad 13: /DETO5 -> /IO_48
- J12 pad 14: /DETO6 -> /IO_46
- J12 pad 15: /USER_IO4 -> /IO_47
- J12 pad 16: /SS2_FPGA -> /IO_75
- J12 pad 17: /MOSI -> /IO_76
- J12 pad 18: /MISO -> /IO_78
- J12 pad 19: /SCK -> /IO_77
- J12 pad 2: /DETO6 -> /IO_51
- J12 pad 20: /RGB_B5 -> /IO_79
- J12 pad 21: /RGB_B3 -> /IO_74
- J12 pad 22: /RGB_B4 -> /IO_80
- J12 pad 23: /RGB_B2 -> /IO_67
- J12 pad 24: /I2S_LRCK -> /IO_63
- J12 pad 25: /I2S_BCK -> /IO_66
- J12 pad 26: /I2S_DIN -> /IO_71
- J12 pad 27: /VSYNC -> /IO_55
- J12 pad 28: /AUDIO_IN -> /IO_54
- J12 pad 29: /3V3mi -> Net-(J12-Pad29)
- J12 pad 3: /DETO3 -> /IO_52
- J12 pad 31: /LED_Y -> /IO_72
- J12 pad 32: /HSYNC -> /IO_59
- J12 pad 33: /RGB_R5 -> /IO_73
- J12 pad 34: /RGB_G5 -> /IO_56
- J12 pad 35: /RGB_R4 -> /IO_57
- J12 pad 36: /RGB_G4 -> /IO_58
- J12 pad 37: /RGB_R3 -> /IO_37
- J12 pad 38: /RGB_G3 -> /IO_38
- J12 pad 39: /RGB_R2 -> /IO_39
- J12 pad 4: /DETO4 -> /IO_53
- J12 pad 40: /RGB_G2 -> /IO_40
- J12 pad 5: /DETO1 -> /IO_41
- J12 pad 6: /FPGA_Tx -> /IO_42
- J12 pad 7: /DETO2 -> /IO_49
- J12 pad 8: /USER_IO2 -> /IO_45
- J12 pad 9: /USER_IO1 -> /IO_44
- J13 pad 1: /SS2_FPGA -> /IO_17
- J13 pad 10: /DETO4 -> /IO_24
- J13 pad 2: /MOSI -> /IO_18
- J13 pad 3: /MISO -> /IO_19
- J13 pad 4: /SCK -> /IO_20
- J13 pad 7: /DETO1 -> /IO_21
- J13 pad 8: /DETO2 -> /IO_22
- J13 pad 9: /DETO3 -> /IO_23
- J14 pad 2: Net-(J14-Pad2) -> unconnected-(J14-Pad2)
- J14 pad 6: Net-(J14-Pad6) -> unconnected-(J14-Pad6)
- J15 pad 1: +5V -> +3V3
- J15 pad 2: /D- -> GND
- J15 pad 3: /D+ -> /IO_63
- J15 pad 4: GND -> /IO_71
- J15 pad 5: /RX- -> /IO_66
- J15 pad 6: /RX+ -> /IO_73
- J16 pad 1: /AUDIO_IN -> /IO_37
- J16 pad 2: /I2S_BCK -> /IO_38
- J16 pad 3: /I2S_DIN -> /IO_39
- J16 pad 4: /I2S_LRCK -> /IO_40
- J17 pad 2: /DETO1 -> /IO_41
- J17 pad 3: /FPGA_Tx -> /IO_42
- R1 pad 1: /DETO5 -> /IO_50
- R10 pad 1: /DETO5 -> /IO_80
- R10 pad 2: /RX- -> Net-(P1-PadCD)
- R2 pad 1: /DETO6 -> /IO_51
- R5 pad 1: /DETO3 -> GND
- R5 pad 2: Net-(J14-Pad6) -> Net-(BUT1-Pad1)
- R6 pad 1: /DETO4 -> GND
- R6 pad 2: Net-(J14-Pad2) -> Net-(BUT2-Pad1)
- R7 pad 1: /DETO2 -> GND
- R7 pad 2: /TX+b -> Net-(D5-Pad1)
- R8 pad 1: /USER_IO1 -> GND
- R8 pad 2: /D- -> Net-(D6-Pad1)
- R9 pad 1: /USER_IO0 -> GND
- R9 pad 2: /D+ -> Net-(D7-Pad1)
Other:
- board size 112.4 x 105.5 mm -> 150.5 x 105.5 mm
- board text added: "DB9"
- board text added: "I2C DISPLAY"
- board text added: "I2S PCM5102"
- board text added: "MISTER MODULE"
- board text added: "POSEIDON BUS"
- board text added: "PS2 KEYB"
- board text added: "PS2 MOUSE"
- board text added: "ROTATIVE ENCODER"
- board text added: "SD"
- board text added: "TERASIC BUS"
- board text removed: "PS2"
- board text removed: "STANDALONE BOARD ================ 2 PMOD VIDEO 1 PMOD SDCARD 1 DETO AUDIO 1 USB3 JOYSTICK 1 PS2 KEYB&MOUSE 1 UART"
- board text removed: "TERASIC 2x20"
- board text removed: "USB3 NEEDS EXTERNAL LEVEL SHIFTER"

Commit message: updated WIP
Parts:
- added J22: PMOD5, footprints:PMOD_Female_Horizontal_2, F.Cu at (196.8, 36.2)
- added J23: Conn_02x20_Odd_Even, Connector_PinHeader_2.54mm:PinHeader_2x20_P2.54mm_Vertical, F.Cu at (49.5, 70.5)
- J17: value Conn_01x03 -> Conn_01x05; footprint Connector_PinHeader_2.54mm:PinHeader_1x03_P2.54mm_Vertical -> Connector_PinSocket_2.54mm:PinSocket_1x05_P2.54mm_Vertical
- J4: value Conn_02x20_Odd_Even -> Conn_01x06; footprint Connector_PinHeader_2.54mm:PinHeader_2x20_P2.54mm_Vertical -> footprints:PCM5102
- moved J12 83.0 mm to (49.5, 123.8), turned to 180 degrees
- moved J4 36.3 mm to (87.0, 73.0), turned to 90 degrees
- moved J5 34.7 mm to (55.2, 83.8), turned to 180 degrees
- moved JP2 15.5 mm to (58.4, 91.4)
- moved JP1 14.2 mm to (58.4, 101.6)
- moved J17 2.30 mm to (97.2, 123.8)
Connections:
- BUT1 pad 2: /IO_57 -> /IO_49
- BUT2 pad 2: /IO_58 -> /IO_50
- D1 pad 1: /IO_50 -> /IO_79
- D2 pad 1: /IO_51 -> /IO_80
- D3 pad 1: /IO_52 -> /IO_77
- D4 pad 1: /IO_53 -> /IO_78
- D5 pad 2: /IO_72 -> /IO_53
- D6 pad 2: /IO_41 -> /IO_54
- D7 pad 2: /IO_73 -> /IO_51
- J11 pad 10: /IO_65 -> /IO_47
- J11 pad 11: /IO_57 -> /IO_49
- J11 pad 12: /IO_66 -> /IO_57
- J11 pad 13: /IO_58 -> /IO_50
- J11 pad 15: /IO_59 -> /IO_54
- J11 pad 16: /IO_67 -> /IO_59
- J11 pad 18: /IO_68 -> /IO_49
- J11 pad 19: /IO_60 -> /IO_48
- J11 pad 21: /IO_61 -> /IO_45
- J11 pad 22: /IO_69 -> /IO_52
- J11 pad 23: /IO_62 -> /IO_46
- J11 pad 24: /IO_70 -> /IO_47
- J11 pad 3: /IO_54 -> /IO_56
- J11 pad 35: /IO_63 -> /IO_60
- J11 pad 40: /IO_71 -> /IO_58
- J11 pad 7: /IO_56 -> /IO_52
- J11 pad 8: /IO_64 -> /IO_48
- J12 pad 1: /IO_50 -> /IO_79
- J12 pad 10: /IO_43 -> /IO_72
- J12 pad 13: /IO_48 -> /IO_69
- J12 pad 14: /IO_46 -> /IO_70
- J12 pad 15: /IO_47 -> /IO_67
- J12 pad 16: /IO_75 -> /IO_68
- J12 pad 17: /IO_76 -> /IO_65
- J12 pad 18: /IO_78 -> /IO_66
- J12 pad 19: /IO_77 -> /IO_63
- J12 pad 2: /IO_51 -> /IO_80
- J12 pad 20: /IO_79 -> /IO_64
- J12 pad 21: /IO_74 -> /IO_61
- J12 pad 22: /IO_80 -> /IO_62
- J12 pad 23: /IO_67 -> /IO_59
- J12 pad 24: /IO_63 -> /IO_60
- J12 pad 25: /IO_66 -> /IO_57
- J12 pad 26: /IO_71 -> /IO_58
- J12 pad 28: /IO_54 -> /IO_56
- J12 pad 3: /IO_52 -> /IO_77
- J12 pad 31: /IO_72 -> /IO_53
- J12 pad 32: /IO_59 -> /IO_54
- J12 pad 33: /IO_73 -> /IO_51
- J12 pad 34: /IO_56 -> /IO_52
- J12 pad 35: /IO_57 -> /IO_49
- J12 pad 36: /IO_58 -> /IO_50
- J12 pad 37: /IO_37 -> /IO_47
- J12 pad 38: /IO_38 -> /IO_48
- J12 pad 39: /IO_39 -> /IO_45
- J12 pad 4: /IO_53 -> /IO_78
- J12 pad 40: /IO_40 -> /IO_46
- J12 pad 5: /IO_41 -> /IO_75
- J12 pad 6: /IO_42 -> /IO_76
- J12 pad 7: /IO_49 -> /IO_73
- J12 pad 8: /IO_45 -> /IO_74
- J12 pad 9: /IO_44 -> /IO_71
- J15 pad 1: +3V3 -> /IO_51
- J15 pad 2: GND -> /IO_57
- J15 pad 3: /IO_63 -> /IO_58
- J15 pad 4: /IO_71 -> /IO_60
- J15 pad 5: /IO_66 -> GND
- J15 pad 6: /IO_73 -> +3V3
- J16 pad 1: /IO_37 -> /IO_47
- J16 pad 10: /IO_73 -> /IO_52
- J16 pad 2: /IO_38 -> /IO_48
- J16 pad 3: /IO_39 -> /IO_45
- J16 pad 4: /IO_40 -> /IO_46
- J16 pad 7: /IO_63 -> /IO_54
- J16 pad 8: /IO_71 -> /IO_59
- J16 pad 9: /IO_66 -> /IO_49
- J17 pad 2: /IO_41 -> /IO_75
- J17 pad 3: /IO_42 -> /IO_76
- J4 pad 1: /IO_1 -> /IO_57
- J4 pad 2: /IO_2 -> /IO_58
- J4 pad 3: /IO_3 -> /IO_60
- J4 pad 4: /IO_4 -> /IO_51
- J4 pad 5: /IO_5 -> GND
- J4 pad 6: /IO_6 -> +3V3
- J5 pad 1: /IO_72 -> /IO_42
- J5 pad 2: /IO_39 -> /IO_43
- J5 pad 3: /IO_40 -> /IO_44
- J7 pad 1: /IO_59 -> /IO_54
- J7 pad 2: /IO_67 -> /IO_59
- J7 pad 3: /IO_56 -> /IO_52
- J8 pad 4: /IO_54 -> /IO_56
- JP1 pad 2: Net-(J4-Pad11) -> Net-(J23-Pin_11)
- JP2 pad 2: Net-(J4-Pad29) -> Net-(J23-Pin_29)
- R1 pad 1: /IO_50 -> /IO_79
- R10 pad 1: /IO_80 -> /IO_62
- R14 pad 1: /IO_52 -> /IO_77
- R15 pad 1: /IO_53 -> /IO_78
- R2 pad 1: /IO_51 -> /IO_80
- RN2 pad 5: /IO_76 -> /IO_65
- RN2 pad 6: /IO_80 -> /IO_62
- RN2 pad 7: /IO_77 -> /IO_63
- RN2 pad 8: /IO_78 -> /IO_66
- RN3 pad 5: /IO_79 -> /IO_64
- RN3 pad 6: /IO_74 -> /IO_61
- RN3 pad 7: /IO_75 -> /IO_68
- U2 pad 3: /IO_49 -> /IO_73
- U2 pad 4: /IO_46 -> /IO_70
- U2 pad 5: /IO_48 -> /IO_69
- U2 pad 6: /IO_47 -> /IO_67
- U2 pad 7: /IO_43 -> /IO_72
- U2 pad 8: /IO_45 -> /IO_74
- U2 pad 9: /IO_44 -> /IO_71
