File: psd_bus.kicad_sch (KiCad schematic)
At the start: 70 parts, among them J1 PMOD1, J10 PMOD2, J11 RASPBERRYPI_BPLUS_BONNETNODIM, J12 Conn_02x20_Odd_Even, J13 PMOD3, J14 DINC_MIN_TM_6_1, J15 Conn_01x06, J16 PMOD2, J17 Conn_01x03, J18 DINC_MIN_TM_6_1, J19 Conn_02x06_Odd_Even, J2 Conn_02x40_Odd_Even, J20 USB3_A, J21 DB9_Male_MountingHoles, J3 PMOD3, J4 Conn_02x20_Odd_Even, J5 Conn_01x03, J6 Conn_01x02, J7 Conn_01x05, J8 Conn_01x04, J9 Conn_01x02, P1 MEM1055-00-280-01-B, U1 LM1117-3.3, U2 TXS0108EPWR

Commit message: preliminary distribution on pcb
Parts:
- D5, D6, D7: footprint (none) -> LED_SMD:LED_0805_2012Metric_Pad1.15x1.40mm_HandSolder
- J15: footprint gomaDOSzero:PCM5102 -> footprints:PCM5102
- J16: value PMOD2 -> PMOD5
- J18: footprint ps2:DINC_MIN_TM_6_1PRIMARY -> footprints:DINC_MIN_TM_6_1PRIMARY
- J20: footprint varis:USB-3.0-TH_C69073 -> footprints:USB-3.0-TH_C69073; old_FP Connector_USB:USB3_A_Molex_48393-001 -> (none)
- J3: value PMOD3 -> PMOD4
- J8: footprint gomaDOSzero:I2C_DISPLAY_MULTI2 -> footprints:I2C_DISPLAY_MULTI2
- P1: footprint Componentes:GCT_MEM1055-00-280-01-B -> Connector_Card:SD_TE_2041021
- RN2, RN3: footprint Componentes:Array0603 -> Resistor_SMD:R_Array_Concave_4x0603
Changed lines of the file:
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@@
     (property "Reference" "D6" (id 0) (at 247.396 181.61 0))
     (property "Value" "LED" (id 1) (at 251.46 181.61 0))
-    (property "Footprint" "" (id 2) (at 251.46 184.404 0)
+    (property "Footprint" "LED_SMD:LED_0805_2012Metric_Pad1.15x1.40mm_HandSolder" (id 2) (at 251.46 184.404 0)
       (effects (font (size 1.27 1.27)) hide)
     )
@@
     (property "Reference" "RN2" (id 0) (at 187.839 217.17 0))
     (property "Value" "20K" (id 1) (at 187.839 219.4814 0))
-    (property "Footprint" "Componentes:Array0603" (id 2) (at 187.839 220.345 0)
+    (property "Footprint" "Resistor_SMD:R_Array_Concave_4x0603" (id 2) (at 187.839 220.345 0)
       (effects (font (size 1.27 1.27)) hide)
     )
@@
       (effects (font (size 1.27 1.27)) (justify right))
     )
-    (property "Footprint" "varis:USB-3.0-TH_C69073" (id 2) (at 378.46 91.44 0)
+    (property "Footprint" "footprints:USB-3.0-TH_C69073" (id 2) (at 378.46 91.44 0)
       (effects (font (size 1.27 1.27)) hide)
     )
@@
       (effects (font (size 1.27 1.27)) hide)
     )
-    (property "old_FP" "Connector_USB:USB3_A_Molex_48393-001" (id 4) (at 382.27 93.98 0)
+    (property "old_FP" "" (id 4) (at 382.27 93.98 0)
       (effects (font (size 1.27 1.27)) hide)
     )
@@
     (in_bom yes) (on_board yes)
     (property "Reference" "J3" (id 0) (at 200.66 64.3382 0))
-    (property "Value" "PMOD3" (id 1) (at 200.66 66.6496 0))
+    (property "Value" "PMOD4" (id 1) (at 200.66 66.6496 0))
     (property "Footprint" "footprints:PMOD_Female_Horizontal_2" (id 2) (at 199.39 74.93 0)
       (effects (font (size 1.27 1.27)) hide)
@@
     (property "Reference" "D5" (id 0) (at 247.396 174.244 0))
     (property "Value" "LED" (id 1) (at 251.206 174.244 0))
-    (property "Footprint" "" (id 2) (at 251.46 177.038 0)
+    (property "Footprint" "LED_SMD:LED_0805_2012Metric_Pad1.15x1.40mm_HandSolder" (id 2) (at 251.46 177.038 0)
       (effects (font (size 1.27 1.27)) hide)
     )
@@
     (property "Reference" "P1" (id 0) (at 245.364 224.4852 0))
     (property "Value" "MEM1055-00-280-01-B" (id 1) (at 245.364 226.7966 0))
-    (property "Footprint" "Componentes:GCT_MEM1055-00-280-01-B" (id 2) (at 245.364 251.587 0)
+    (property "Footprint" "Connector_Card:SD_TE_2041021" (id 2) (at 245.364 251.587 0)
       (effects (font (size 1.27 1.27)) (justify left bottom) hide)
     )
@@
       (effects (font (size 1.27 1.27)) (justify left))
     )
-    (property "Footprint" "gomaDOSzero:PCM5102" (id 2) (at 268.224 75.184 0)
+    (property "Footprint" "footprints:PCM5102" (id 2) (at 268.224 75.184 0)
       (effects (font (size 1.27 1.27)) hide)
     )
@@
       (effects (font (size 1.778 1.5113)) (justify right))
     )
-    (property "Footprint" "ps2:DINC_MIN_TM_6_1PRIMARY" (id 2) (at 374.65 233.172 0)
+    (property "Footprint" "footprints:DINC_MIN_TM_6_1PRIMARY" (id 2) (at 374.65 233.172 0)
       (effects (font (size 1.27 1.27)) hide)
     )
@@
     (property "Reference" "RN3" (id 0) (at 187.706 200.152 0))
     (property "Value" "20K" (id 1) (at 187.706 202.4634 0))
-    (property "Footprint" "Componentes:Array0603" (id 2) (at 187.706 203.327 0)
+    (property "Footprint" "Resistor_SMD:R_Array_Concave_4x0603" (id 2) (at 187.706 203.327 0)
       (effects (font (size 1.27 1.27)) hide)
     )
@@
     (property "Reference" "D7" (id 0) (at 247.396 189.23 0))
     (property "Value" "LED" (id 1) (at 251.46 189.23 0))
-    (property "Footprint" "" (id 2) (at 251.46 192.024 0)
+    (property "Footprint" "LED_SMD:LED_0805_2012Metric_Pad1.15x1.40mm_HandSolder" (id 2) (at 251.46 192.024 0)
       (effects (font (size 1.27 1.27)) hide)
     )
@@
   (symbol (lib_id "Connector_Generic:Conn_02x06_Top_Bottom") (at 256.794 33.02 0) (unit 1)
     (in_bom yes) (on_board yes) (fields_autoplaced)
-    (property "Reference" "J16" (id 0) (at 258.064 20.955 0))
-    (property "Value" "PMOD2" (id 1) (at 258.064 23.495 0))
+    (property "Reference" "J16" (id 0) (at 258.064 21.59 0))
+    (property "Value" "PMOD5" (id 1) (at 258.064 24.13 0))
     (property "Footprint" "footprints:PMOD_Female_Horizontal_2" (id 2) (at 256.794 33.02 0)
       (effects (font (size 1.27 1.27)) hide)
@@
       (effects (font (size 1.27 1.27)) (justify left))
     )
-    (property "Footprint" "gomaDOSzero:I2C_DISPLAY_MULTI2" (id 2) (at 94.234 151.384 0)
+    (property "Footprint" "footprints:I2C_DISPLAY_MULTI2" (id 2) (at 94.234 151.384 0)
       (effects (font (size 1.27 1.27)) hide)
     )
@@
     )
     (path "/22ef7ca9-8c9f-4920-b661-b81bb0bbee20"
-      (reference "D5") (unit 1) (value "LED") (footprint "")
+      (reference "D5") (unit 1) (value "LED") (footprint "LED_SMD:LED_0805_2012Metric_Pad1.15x1.40mm_HandSolder")
     )
     (path "/01ee5666-fe7b-4368-a990-0645b8571000"
-      (reference "D6") (unit 1) (value "LED") (footprint "")
+      (reference "D6") (unit 1) (value "LED") (footprint "LED_SMD:LED_0805_2012Metric_Pad1.15x1.40mm_HandSolder")
     )
     (path "/a09733a9-f405-499d-8c26-78b234999d34"
-      (reference "D7") (unit 1) (value "LED") (footprint "")
+      (reference "D7") (unit 1) (value "LED") (footprint "LED_SMD:LED_0805_2012Metric_Pad1.15x1.40mm_HandSolder")
     )
     (path "/a69b7b01-ac9d-420b-b658-6c6a0976ffbd"
@@
     )
     (path "/214e3cb8-319d-4835-b5ba-372ad4fb3113"
-      (reference "J3") (unit 1) (value "PMOD3") (footprint "footprints:PMOD_Female_Horizontal_2")
+      (reference "J3") (unit 1) (value "PMOD4") (footprint "footprints:PMOD_Female_Horizontal_2")
     )
     (path "/e0abf8f3-23af-4028-aae2-bcb687774a16"
@@
     )
     (path "/c71fd0a8-53e1-417d-9543-665bdfd8272f"
-      (reference "J8") (unit 1) (value "Conn_01x04") (footprint "gomaDOSzero:I2C_DISPLAY_MULTI2")
+      (reference "J8") (unit 1) (value "Conn_01x04") (footprint "footprints:I2C_DISPLAY_MULTI2")
     )
     (path "/e383b838-ec38-43e6-ba3f-d4d24bed37e7"
@@
     )
     (path "/4ac0b295-841a-4940-8973-8536013f104c"
-      (reference "J15") (unit 1) (value "Conn_01x06") (footprint "gomaDOSzero:PCM5102")
+      (reference "J15") (unit 1) (value "Conn_01x06") (footprint "footprints:PCM5102")
     )
     (path "/a3f53ab1-4eba-45f1-83ea-971ce25e0ad4"
-      (reference "J16") (unit 1) (value "PMOD2") (footprint "footprints:PMOD_Female_Horizontal_2")
+      (reference "J16") (unit 1) (value "PMOD5") (footprint "footprints:PMOD_Female_Horizontal_2")
     )
     (path "/c4420e99-4bbc-4042-9222-5779846eccc4"
@@
     )
     (path "/5cee05e3-80b0-4c59-82b6-84b4d9eb09c1"
-      (reference "J18") (unit 1) (value "DINC_MIN_TM_6_1") (footprint "ps2:DINC_MIN_TM_6_1PRIMARY")
+      (reference "J18") (unit 1) (value "DINC_MIN_TM_6_1") (footprint "footprints:DINC_MIN_TM_6_1PRIMARY")
     )
     (path "/b4d677b3-303f-45f7-ae81-8eee1c071e02"
@@
     )
     (path "/1391764e-17ca-4a9e-a2dc-f725e9540aba"
-      (reference "J20") (unit 1) (value "USB3_A") (footprint "varis:USB-3.0-TH_C69073")
+      (reference "J20") (unit 1) (value "USB3_A") (footprint "footprints:USB-3.0-TH_C69073")
     )
     (path "/dd28f949-8cdb-433b-b7a3-c05902a67e58"
@@
     )
     (path "/23296ebb-694d-4659-8c27-83a176b90810"
-      (reference "P1") (unit 1) (value "MEM1055-00-280-01-B") (footprint "Componentes:GCT_MEM1055-00-280-01-B")
+      (reference "P1") (unit 1) (value "MEM1055-00-280-01-B") (footprint "Connector_Card:SD_TE_2041021")
     )
     (path "/2835995c-2375-46e5-9b30-f9aa5106ba72"
@@
     )
     (path "/0b87fef1-c8b2-4710-9574-5524d82fe245"
-      (reference "RN2") (unit 1) (value "20K") (footprint "Componentes:Array0603")
+      (reference "RN2") (unit 1) (value "20K") (footprint "Resistor_SMD:R_Array_Concave_4x0603")
     )
     (path "/827cfeed-10e1-49ff-9a37-c3aeec114ef2"
-      (reference "RN3") (unit 1) (value "20K") (footprint "Componentes:Array0603")
+      (reference "RN3") (unit 1) (value "20K") (footprint "Resistor_SMD:R_Array_Concave_4x0603")
     )
     (path "/7e8d0e61-a648-4421-a958-e042a87d1564"

Commit message: updated WIP
Parts:
- removed J17: Conn_01x03, Connector_PinHeader_2.54mm:PinHeader_1x03_P2.54mm_Vertical, symbol Connector_Generic:Conn_01x03
- removed J4: Conn_02x20_Odd_Even, Connector_PinHeader_2.54mm:PinHeader_2x20_P2.54mm_Vertical, symbol Connector_Generic:Conn_02x20_Odd_Even
- added J17: Conn_01x05, Connector_PinSocket_2.54mm:PinSocket_1x05_P2.54mm_Vertical, symbol Connector_Generic:Conn_01x05
- added J22: PMOD5, footprints:PMOD_Female_Horizontal_2, symbol Connector_Generic:Conn_02x06_Top_Bottom
- added J23: Conn_02x20_Odd_Even, Connector_PinHeader_2.54mm:PinHeader_2x20_P2.54mm_Vertical, symbol Connector_Generic:Conn_02x20_Odd_Even
- added J4: Conn_01x06, footprints:PCM5102, symbol Connector_Generic:Conn_01x06
Connections:
- net +3V3: now also J15.6 (Pin_6), J22.12 (Pin_12), J22.6 (Pin_6), J4.6 (Pin_6); no longer J15.1 (Pin_1)
- net GND: now also J15.5 (Pin_5), J17.1 (Pin_1), J22.11 (Pin_11), J22.5 (Pin_5), J23.12 (Pin_12), J23.30 (Pin_30), J4.5 (Pin_5); no longer J15.2 (Pin_2)
- net IO_1: now also J23.39 (Pin_39)
- net IO_10: now also J23.32 (Pin_32)
- net IO_11: now also J23.27 (Pin_27)
- net IO_12: now also J23.28 (Pin_28)
- net IO_13: now also J23.25 (Pin_25)
- net IO_14: now also J23.26 (Pin_26)
- net IO_15: now also J23.23 (Pin_23)
- net IO_16: now also J23.24 (Pin_24)
- net IO_17: now also J23.21 (Pin_21)
- net IO_18: now also J23.22 (Pin_22)
- net IO_19: now also J23.19 (Pin_19)
- net IO_2: now also J23.40 (Pin_40)
- net IO_20: now also J23.20 (Pin_20)
- net IO_21: now also J23.17 (Pin_17)
- net IO_22: now also J23.18 (Pin_18)
- net IO_23: now also J23.15 (Pin_15)
- net IO_24: now also J23.16 (Pin_16)
- net IO_25: now also J23.13 (Pin_13)
- net IO_26: now also J23.14 (Pin_14)
- net IO_27: now also J23.9 (Pin_9)
- net IO_28: now also J23.10 (Pin_10)
- net IO_29: now also J23.7 (Pin_7)
- net IO_3: now also J23.37 (Pin_37)
- net IO_30: now also J23.8 (Pin_8)
- net IO_31: now also J23.5 (Pin_5)
- net IO_32: now also J23.6 (Pin_6)
- net IO_37: now also J22.1 (Pin_1), J23.3 (Pin_3); no longer J12.37 (Pin_37), J16.1 (Pin_1)
- net IO_38: now also J22.2 (Pin_2), J23.4 (Pin_4); no longer J12.38 (Pin_38), J16.2 (Pin_2)
- net IO_39: now also J22.3 (Pin_3), J23.1 (Pin_1); no longer J12.39 (Pin_39), J16.3 (Pin_3), J5.2 (Pin_2)
- net IO_4: now also J23.38 (Pin_38)
- net IO_40: now also J22.4 (Pin_4), J23.2 (Pin_2); no longer J12.40 (Pin_40), J16.4 (Pin_4), J5.3 (Pin_3)
- net IO_41: now also J22.7 (Pin_7); no longer D6.2 (A), J12.5 (Pin_5)
- net IO_42: now also J5.1 (Pin_1), J22.8 (Pin_8); no longer J12.6 (Pin_6)
- net IO_43: now also J5.2 (Pin_2), J22.9 (Pin_9); no longer J12.10 (Pin_10), U2.7 (A6)
- net IO_44: now also J5.3 (Pin_3), J22.10 (Pin_10); no longer J12.9 (Pin_9), U2.9 (A8)
- net IO_45: now also J11.21 (SPI_MISO), J12.39 (Pin_39), J16.3 (Pin_3); no longer J12.8 (Pin_8), U2.8 (A7)
- net IO_46: now also J11.23 (SPI_SCLK), J12.40 (Pin_40), J16.4 (Pin_4); no longer J12.14 (Pin_14), U2.4 (A3)
- net IO_47: now also J11.10 (RXD), J11.24 (#SPI_CE0), J12.37 (Pin_37), J16.1 (Pin_1); no longer J12.15 (Pin_15), U2.6 (A5)
- net IO_48: now also J11.19 (SPI_MOSI), J11.8 (TXD), J12.38 (Pin_38), J16.2 (Pin_2); no longer J12.13 (Pin_13), U2.5 (A4)
- net IO_49: now also BUT1.2, J11.11 (GPIO17), J11.18 (GPIO24), J12.35 (Pin_35), J16.9 (Pin_9); no longer J12.7 (Pin_7), U2.3 (A2)
- net IO_5: now also J23.35 (Pin_35)
- net IO_50: now also BUT2.2, J11.13 (GPIO27), J12.36 (Pin_36); no longer D1.1 (K), J12.1 (Pin_1), R1.1
- net IO_51: now also D7.2 (A), J12.33 (Pin_33), J15.1 (Pin_1), J4.4 (Pin_4); no longer D2.1 (K), J12.2 (Pin_2), R2.1
- net IO_52: now also J11.22 (GPIO25), J11.7 (GPIO4), J12.34 (Pin_34), J16.10 (Pin_10), J7.3 (Pin_3); no longer D3.1 (K), J12.3 (Pin_3), R14.1
- net IO_53: now also D5.2 (A), J12.31 (Pin_31), J17.4 (Pin_4); no longer D4.1 (K), J12.4 (Pin_4), R15.1
- net IO_54: now also D6.2 (A), J11.15 (GPIO22), J12.32 (Pin_32), J16.7 (Pin_7), J7.1 (Pin_1), J17.5 (Pin_5); no longer J11.3 (SDA), J12.28 (Pin_28), J8.4 (Pin_4)
- net IO_56: now also J11.3 (SDA), J12.28 (Pin_28), J8.4 (Pin_4); no longer J11.7 (GPIO4), J12.34 (Pin_34), J7.3 (Pin_3)
- net IO_57: now also J11.12 (GPIO18), J12.25 (Pin_25), J15.2 (Pin_2), J4.1 (Pin_1); no longer BUT1.2, J11.11 (GPIO17), J12.35 (Pin_35)
- net IO_58: now also J11.40 (GPIO21), J12.26 (Pin_26), J15.3 (Pin_3), J4.2 (Pin_2); no longer BUT2.2, J11.13 (GPIO27), J12.36 (Pin_36)
- net IO_59: now also J11.16 (GPIO23), J12.23 (Pin_23), J16.8 (Pin_8), J7.2 (Pin_2); no longer J11.15 (GPIO22), J12.32 (Pin_32), J7.1 (Pin_1)
- net IO_6: now also J23.36 (Pin_36)
- net IO_60: now also J11.35 (GPIO19), J12.24 (Pin_24), J15.4 (Pin_4), J4.3 (Pin_3); no longer J11.19 (SPI_MOSI)
- net IO_61: now also J12.21 (Pin_21), P1.P9 (DAT2), RN3.6; no longer J11.21 (SPI_MISO)
- net IO_62: now also J12.22 (Pin_22), R10.1, RN2.6; no longer J11.23 (SPI_SCLK)
- net IO_63: now also J12.19 (Pin_19), P1.P5 (CLK), RN2.7; no longer J11.35 (GPIO19), J12.24 (Pin_24), J15.3 (Pin_3), J16.7 (Pin_7)
- net IO_64: now also J12.20 (Pin_20), P1.P8 (DAT1), RN3.5; no longer J11.8 (TXD)
- net IO_65: now also J12.17 (Pin_17), P1.P2 (CMD), RN2.5; no longer J11.10 (RXD)
- net IO_66: now also J12.18 (Pin_18), P1.P7 (DAT0), RN2.8; no longer J11.12 (GPIO18), J12.25 (Pin_25), J15.5 (Pin_5), J16.9 (Pin_9)
- net IO_67: now also J12.15 (Pin_15), U2.6 (A5); no longer J11.16 (GPIO23), J12.23 (Pin_23), J7.2 (Pin_2)
- net IO_68: now also J12.16 (Pin_16), P1.P1 (DAT3), RN3.7; no longer J11.18 (GPIO24)
- net IO_69: now also J12.13 (Pin_13), U2.5 (A4); no longer J11.22 (GPIO25)
- net IO_7: now also J23.33 (Pin_33)
- net IO_70: now also J12.14 (Pin_14), U2.4 (A3); no longer J11.24 (#SPI_CE0)
- net IO_71: now also J12.9 (Pin_9), U2.9 (A8); no longer J11.40 (GPIO21), J12.26 (Pin_26), J15.4 (Pin_4), J16.8 (Pin_8)
- net IO_72: now also J12.10 (Pin_10), U2.7 (A6); no longer D5.2 (A), J12.31 (Pin_31), J5.1 (Pin_1)
- net IO_73: now also J12.7 (Pin_7), U2.3 (A2); no longer D7.2 (A), J12.33 (Pin_33), J15.6 (Pin_6), J16.10 (Pin_10)
- net IO_74: now also J12.8 (Pin_8), U2.8 (A7); no longer J12.21 (Pin_21), P1.P9 (DAT2), RN3.6
- net IO_75: now also J12.5 (Pin_5), J17.2 (Pin_2); no longer J12.16 (Pin_16), P1.P1 (DAT3), RN3.7
- net IO_76: now also J12.6 (Pin_6), J17.3 (Pin_3); no longer J12.17 (Pin_17), P1.P2 (CMD), RN2.5
- net IO_77: now also D3.1 (K), J12.3 (Pin_3), R14.1; no longer J12.19 (Pin_19), P1.P5 (CLK), RN2.7
- net IO_78: now also D4.1 (K), J12.4 (Pin_4), R15.1; no longer J12.18 (Pin_18), P1.P7 (DAT0), RN2.8
- net IO_79: now also D1.1 (K), J12.1 (Pin_1), R1.1; no longer J12.20 (Pin_20), P1.P8 (DAT1), RN3.5
- net IO_8: now also J23.34 (Pin_34)
- net IO_80: now also D2.1 (K), J12.2 (Pin_2), R2.1; no longer J12.22 (Pin_22), R10.1, RN2.6
- net IO_9: now also J23.31 (Pin_31)
- net at JP2.2 (Pin_2): now also J23.29 (Pin_29)
- net at JP1.2 (Pin_2): now also J23.11 (Pin_11)
Other:
- note added: "(***)"
- note added: "AUDIO_L"
- note added: "AUDIO_R"
- note added: "AUDIO_SPDIF"
- note added: "BTN_OSD"
- note added: "BTN_RESET"
- note added: "BTN_USER"
- note added: "I2S_MCLK"
- note added: "MIDI_OUT"
- note added: "PMOD 1"
- note added: "PMOD 2"
- note added: "PMOD 5"
- note added: "PMOD 5 WITH TERASIC CONN. ============================= PMOD 1/2/5 WITH MISTER MODULE RPI CONN. WITH MISTER MODULE AND PIMIDI PMOD 5 WITH PMOD I2S LED USER WITH MISTER MODULE LED POWER WITH PMOD I2S LED HDD WITH UART RX PIMIDI: DAC I2S, DISPLAY, BUTTONS AND ENCODER"
- note added: "PMOD 6 (*)"
- note added: "PMOD AUDIO (**)"
- note added: "PMOD I2S (**) (PCM5102A)"
- note added: "UART_CTS"
- note added: "UART_RTS"
- note removed: "EXTERNAL MISTER MODULE (*)"
- note removed: "PMOD 1 (*)"
- note removed: "PMOD 1/2/5 WITH MISTER MODULE RPI CONN. WITH MISTER MODULE AND PIMIDI PMOD 5 WITH PMOD I2S LED USER WITH MISTER MODULE LED POWER WITH PMOD I2S LED HDD WITH UART RX PIMIDI: DAC I2S, DISPLAY, BUTTONS AND ENCODER"
- note removed: "PMOD 2 (*)"
- note removed: "PMOD 5 (*)"
- note removed: "PMOD I2S (*) (PCM5102A)"
- moved on the sheet: BUT1, BUT2, C4, D5, D6, D7, J12, J5, J7, J8, JP3, JP4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
